File: hardware/usb.kicad_sch (KiCad schematic)
At the start: 6 parts, among them J2 2137160001, U2 USBLC6-2SC6

Commit message: route USBC connector
Parts:
- removed F1: 500mA, Fuse:Fuse_1206_3216Metric, symbol Device:Polyfuse_Small
- removed USB1: Molex-0548190589, random-keyboard-parts:Molex-0548190589, symbol random-keyboard-parts:Molex-0548190589
Connections:
- net USB_D+: now also U2.6
- net USB_D-: no longer U2.6
- no-connect marks 3 -> 2
